File: Hardware/Kicad_files/Tesi.kicad_sch (KiCad schematic)
At the start: 46 parts, among them IC1 TPS63070RNMR, J1 Ext_power_conn, J2 Bat_conn, J3 Out_conn, Q1 FS8205, Q2 DMP1045U-7, SW1 Power_sw_conn, SW2 Switch_pins, SW3 SW_DIP_x02, U1 DW01A, U2 MCP73831-2-OT

Commit message: Update
Other:
- note added: "Pull-down resistor when VBUS unplugged"
- note removed: "Pull-down resistor when USB unplugged"
Changed lines of the file:
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@@
 		)
 	)
-	(text "Pull-down resistor\nwhen USB unplugged"
+	(text "Pull-down resistor\nwhen VBUS unplugged"
 		(exclude_from_sim no)
-		(at 18.288 146.05 0)
+		(at 17.018 146.05 0)
 		(effects
 			(font
