File: Hardware/Kicad_files/Tesi.kicad_pcb (KiCad board)
At the start: 2 copper layers, 50 x 50 mm, 65 parts, among them IC1 TPS63070RNMR, J1 Ext_power_conn, J2 Bat_conn, J3 Out_conn, J4 MCU_conn, Q1 FS8205, Q2 DMP1045U-7, Q4 BSS84, SW1 Power_sw_conn, SW2 Switch_pins, SW3 SW_DIP_x02, U1 DW01A, U2 MCP73831-2-OT, U3 MAX17048G_T10

Commit message: Added library footprint
Parts:
- C1: footprint Capacitor_Tantalum_SMD:CP_EIA-3216-18_Kemet-A -> Library:CP_EIA-3216-18_Kemet-A
- C10, C6: footprint Capacitor_SMD:C_0402_1005Metric -> Library:C_0402_1005Metric
- C11, C12, C13, C14, C2, C7: footprint Capacitor_SMD:C_0603_1608Metric -> Library:C_0603_1608Metric
- C3, C4, C5, C8, C9: footprint Capacitor_SMD:C_0805_2012Metric -> Library:C_0805_2012Metric
- D4, D5: footprint Diode_SMD:D_SMA -> Library:D_SMA
- F1: footprint Fuse:Fuse_1812_4532Metric_Pad1.30x3.40mm_HandSolder -> Library:Fuse_1812_4532Metric_Pad1.30x3.40mm_HandSolder
- G***: footprint Loghi:MAICXEN_logo -> Library:MAICXEN_logo
- G*** (x2): footprint Loghi:UniGe_logo -> Library:UniGe_logo
- H1, H2, H3, H4: footprint MountingHole:MountingHole_2.2mm_M2_DIN965_Pad -> Library:MountingHole_2.2mm_M2_DIN965_Pad
- IC1: footprint TPS63070RNMR:TPS630701RNMR -> Library:TPS630701RNMR
- J1, J2, J3, SW1: footprint KF301:KF3012P -> Library:KF3012P
- J4: footprint TerminalBlock:TerminalBlock_Xinya_XY308-2.54-5P_1x05_P2.54mm_Horizontal -> Library:TerminalBlock_Xinya_XY308-2.54-5P_1x05_P2.54mm_Horizontal
- JP1, JP3, JP4, JP6: footprint Jumper:SolderJumper-2_P1.3mm_Bridged_RoundedPad1.0x1.5mm -> Library:SolderJumper-2_P1.3mm_Bridged_RoundedPad1.0x1.5mm
- JP7: footprint Jumper:SolderJumper-3_P1.3mm_Bridged12_RoundedPad1.0x1.5mm_NumberLabels -> Library:SolderJumper-3_P1.3mm_Bridged12_RoundedPad1.0x1.5mm_NumberLabels
- L1: footprint Inductor_SMD:L_Coilcraft_XxL4020 -> Library:L_Coilcraft_XxL4020
- LED_A1, LED_G1: footprint LED_SMD:LED_0603_1608Metric -> Library:LED_0603_1608Metric
- Q1: footprint FS8205:FS8205 -> Library:FS8205
- Q2: footprint Package_TO_SOT_SMD:SOT-23-GATE -> Library:SOT-23-GATE
- Q4: footprint Package_TO_SOT_SMD:SOT-23 -> Library:SOT-23
- R1, R2, R5, RPROG1, Rmos2: footprint Resistor_SMD:R_0603_1608Metric -> Library:R_0603_1608Metric
- R10, R3: footprint Resistor_SMD:R_0805_2012Metric -> Library:R_0805_2012Metric
- R11, R4, R6, R7, R9: footprint Resistor_SMD:R_0402_1005Metric -> Library:R_0402_1005Metric
- RN1: footprint Resistor_SMD:R_Array_Convex_4x0402 -> Library:R_Array_Convex_4x0402
- SW2: footprint Connector_PinHeader_2.54mm:PinHeader_1x02_P2.54mm_Vertical_SMD_Pin1Left -> Library:PinHeader_1x02_P2.54mm_Vertical_SMD_Pin1Left
- SW3: footprint Button_Switch_SMD:SW_DIP_SPSTx02_Slide_KingTek_DSHP02TS_W7.62mm_P1.27mm -> Library:SW_DIP_SPSTx02_Slide_KingTek_DSHP02TS_W7.62mm_P1.27mm
- TP1, TP3: footprint Connector_Pin:Pin_D0.7mm_L6.5mm_W1.8mm_FlatFork -> Library:Pin_D0.7mm_L6.5mm_W1.8mm_FlatFork
- TP2, TP4, TP6, TP7: footprint TestPoint:TestPoint_Pad_D2.0mm -> Library:TestPoint_Pad_D2.0mm
- U1: footprint Package_TO_SOT_SMD:SOT-23-6 -> Library:SOT-23-6
- U2: footprint Package_TO_SOT_SMD:SOT-23-5 -> Library:SOT-23-5
- U3: footprint MAX17048G_T10:SON50P200X200X80-9N -> Library:SON50P200X200X80-9N
